File: pcb/vertex.sch (KiCad schematic (older format))
At the start: 86 parts, among them U1 ATmega32U2-AU, U2 SRV05-4, X1 Crystal_GND24_Small

Commit message: finalized PCB
Parts:
- added C7, C8: 0.1uF, Capacitor_SMD:C_0805_2012Metric, symbol Device:C_Small
- added D24: D_Small, custom_parts:D_SOT-23_ANK_norm, symbol custom:D_AAK_Small
- added MX46, MX47, MX48, MX49, MX50, MX51, MX52, MX53, MX67: MX-NoLED, MX_Only:MXOnly-1U-NoLED, symbol MX_Alps_Hybrid:MX-NoLED
- added MX54: MX-NoLED, MX_Only:MXOnly-2.75U-ReversedStabilizers-NoLED, symbol MX_Alps_Hybrid:MX-NoLED
- added MX55: MX-NoLED, MX_Only:MXOnly-2.25U-ReversedStabilizers-NoLED, symbol MX_Alps_Hybrid:MX-NoLED
- added MX60: MX-NoLED, MX_Only:MXOnly-2U-NoLED, symbol MX_Alps_Hybrid:MX-NoLED
- added MX66: MX-NoLED, MX_Only:MXOnly-1.25U-NoLED, symbol MX_Alps_Hybrid:MX-NoLED
- added R7, R8: 10k, Resistor_SMD:R_0805_2012Metric, symbol Device:R_Small
- added ROT1: Rotary_Encoder_Switch, Rotary_Encoder:RotaryEncoder_Alps_EC11E-Switch_Vertical_H20mm, symbol Device:Rotary_Encoder_Switch
- D1, D10, D11, D12, D13, D14, D15, D16, D17, D18, D19, D2, D20, D21, D22, D23, D3, D4, D5, D6, D7, D8, D9: footprint custom_parts:D_SOT-23_ANK -> custom_parts:D_SOT-23_ANK_norm; symbol Device:D_Small -> custom:D_AAK_Small
- renumbered C6 to C4, C7 to C5, C5 to C6
Connections:
- net GND: now also C7.1, C8.2, ROT1.C
- net VCC: now also R7.2, R8.1
- net col0: now also MX46.2 (ROW)
- net col1: now also MX47.1 (COL); no longer MX39.1 (COL)
- net col10: now also MX53.2 (ROW), MX66.1 (COL)
- net col11: now also MX60.1 (COL), MX67.1 (COL)
- net col2: now also MX39.1 (COL), MX48.2 (ROW); no longer MX40.1 (COL)
- net col3: now also MX40.1 (COL), MX49.1 (COL)
- net col4: now also MX55.2 (ROW)
- net col6: now also MX42.1 (COL), MX54.2 (ROW)
- net col7: now also MX43.1 (COL), MX50.1 (COL); no longer MX42.1 (COL)
- net col8: now also MX44.1 (COL), MX51.2 (ROW); no longer MX43.1 (COL)
- net col9: now also MX52.1 (COL); no longer MX44.1 (COL)
- net row3: now also D24.1 (K)
- net at D1.2 (A1), MX1.2 (ROW): no longer MX2.2 (ROW)
- net at D2.2 (A1), MX3.2 (ROW): no longer MX4.2 (ROW)
- net at D3.2 (A1), MX5.2 (ROW): no longer MX6.2 (ROW)
- net at D4.2 (A1), MX7.2 (ROW): no longer MX8.2 (ROW)
- net at D5.2 (A1), MX9.2 (ROW): no longer MX10.2 (ROW)
- net at D6.2 (A1), MX11.2 (ROW): no longer MX12.2 (ROW)
- net at MX13.2 (ROW): now also D7.3 (A2); no longer D7.2 (A)
- net at D8.2 (A1), MX15.2 (ROW): no longer MX14.2 (ROW)
- net at D9.2 (A1), MX16.2 (ROW): no longer MX17.2 (ROW)
- net at D10.2 (A1), MX18.2 (ROW): no longer MX19.2 (ROW)
- net at D11.2 (A1), MX20.2 (ROW): no longer MX21.2 (ROW)
- net at D12.2 (A1), MX22.2 (ROW): no longer MX23.2 (ROW)
- net at D13.2 (A1), MX24.2 (ROW): no longer MX25.2 (ROW)
- net at D14.2 (A1), MX26.2 (ROW): no longer MX27.2 (ROW)
- net at D15.2 (A1), MX28.2 (ROW): no longer MX29.2 (ROW)
- net at D16.2 (A1), MX30.2 (ROW): no longer MX31.2 (ROW)
- net at D17.2 (A1), MX32.2 (ROW): no longer MX33.2 (ROW)
- net at D18.2 (A1), MX34.2 (ROW): no longer MX35.2 (ROW)
- net at D19.2 (A1), MX36.2 (ROW): now also MX66.2 (ROW); no longer MX37.2 (ROW)
- net at D21.2 (A1), MX40.2 (ROW): now also MX49.2 (ROW); no longer MX41.2 (ROW)
- net at D23.2 (A1), MX45.2 (ROW): now also MX53.1 (COL); no longer MX44.2 (ROW)
- new net: D1.3 (A2), MX2.2 (ROW)
- new net: D2.3 (A2), MX4.2 (ROW)
- new net: D3.3 (A2), MX6.2 (ROW)
- new net: D4.3 (A2), MX8.2 (ROW)
- new net: D5.3 (A2), MX10.2 (ROW)
- new net: D6.3 (A2), MX12.2 (ROW), MX60.2 (ROW)
- new net: D24.2 (A1), MX42.2 (ROW), MX54.1 (COL)
- new net: D24.3 (A2), MX41.2 (ROW), MX55.1 (COL)
- new net: D20.3 (A2), MX38.2 (ROW), MX46.1 (COL)
- new net: D20.2 (A1), MX47.2 (ROW)
- new net: D21.3 (A2), MX39.2 (ROW), MX48.1 (COL)
- new net: C7.2, R7.1, ROT1.A
- new net: C8.1, R8.2, ROT1.B
- new net: D9.3 (A2), MX17.2 (ROW)
- new net: D10.3 (A2), MX19.2 (ROW)
- new net: D11.3 (A2), MX21.2 (ROW)
- new net: D12.3 (A2), MX23.2 (ROW)
- new net: D8.3 (A2), MX14.2 (ROW)
- new net: D13.3 (A2), MX25.2 (ROW)
- new net: D14.3 (A2), MX27.2 (ROW)
- new net: D15.3 (A2), MX29.2 (ROW)
- new net: D16.3 (A2), MX31.2 (ROW)
- new net: D17.3 (A2), MX33.2 (ROW)
- new net: D18.3 (A2), MX35.2 (ROW)
- new net: D19.3 (A2), MX37.2 (ROW), MX67.2 (ROW)
- new net: D22.3 (A2), MX43.2 (ROW), MX50.2 (ROW)
- new net: D22.2 (A1), MX44.2 (ROW), MX51.1 (COL)
- new net: D23.3 (A2), MX52.2 (ROW)
Other:
- moved on the sheet: MX39, MX40, MX42, MX43, MX44

Commit message: finalize repo layout
Parts:
- removed C7, C8: 0.1uF, Capacitor_SMD:C_0805_2012Metric, symbol Device:C_Small
- removed R7, R8: 10k, Resistor_SMD:R_0805_2012Metric, symbol Device:R_Small
- removed ROT1: Rotary_Encoder_Switch, Rotary_Encoder:RotaryEncoder_Alps_EC11E-Switch_Vertical_H20mm, symbol Device:Rotary_Encoder_Switch
Changed lines of the file:
@@
 Wire Wire Line
 	10100 1250 10100 1500
-$Comp
-L Device:Rotary_Encoder_Switch ROT1
-U 1 1 61399933
-P 5900 4900
-F 0 "ROT1" H 5950 5350 50  0000 C CNN
-F 1 "Rotary_Encoder_Switch" H 6050 5250 50  0000 C CNN
-F 2 "Rotary_Encoder:RotaryEncoder_Alps_EC11E-Switch_Vertical_H20mm" H 5750 5060 50  0001 C CNN
-F 3 "~" H 5900 5160 50  0001 C CNN
-	1    5900 4900
-	1    0    0    -1
-$EndComp
-$Comp
-L power:GND #PWR0101
-U 1 1 6139ABCA
-P 4750 4900
-F 0 "#PWR0101" H 4750 4650 50  0001 C CNN
-F 1 "GND" H 4755 4727 50  0000 C CNN
-F 2 "" H 4750 4900 50  0001 C CNN
-F 3 "" H 4750 4900 50  0001 C CNN
-	1    4750 4900
-	1    0    0    -1
-$EndComp
-$Comp
-L Device:R_Small R8
-U 1 1 613A7BFB
-P 5150 5100
-F 0 "R8" H 5300 5050 50  0000 R CNN
-F 1 "10k" H 5350 5150 50  0000 R CNN
-F 2 "Resistor_SMD:R_0805_2012Metric" H 5150 5100 50  0001 C CNN
-F 3 "~" H 5150 5100 50  0001 C CNN
-F 4 "C17414" H 5150 5100 50  0001 C CNN "LCSC"
-	1    5150 5100
-	-1   0    0    1
-$EndComp
-$Comp
-L Device:R_Small R7
-U 1 1 613A96D6
-P 5150 4700
-F 0 "R7" H 5300 4650 50  0000 R CNN
-F 1 "10k" H 5350 4750 50  0000 R CNN
-F 2 "Resistor_SMD:R_0805_2012Metric" H 5150 4700 50  0001 C CNN
-F 3 "~" H 5150 4700 50  0001 C CNN
-F 4 "C17414" H 5150 4700 50  0001 C CNN "LCSC"
-	1    5150 4700
-	-1   0    0    1
-$EndComp
-$Comp
-L power:VCC #PWR0102
-U 1 1 613DAA9F
-P 4750 4800
-F 0 "#PWR0102" H 4750 4650 50  0001 C CNN
-F 1 "VCC" H 4765 4973 50  0000 C CNN
-F 2 "" H 4750 4800 50  0001 C CNN
-F 3 "" H 4750 4800 50  0001 C CNN
-	1    4750 4800
-	1    0    0    -1
-$EndComp
-$Comp
-L Device:C_Small C8
-U 1 1 613F61F4
-P 5400 5100
-F 0 "C8" H 5492 5146 50  0000 L CNN
-F 1 "0.1uF" H 5492 5055 50  0000 L CNN
-F 2 "Capacitor_SMD:C_0805_2012Metric" H 5400 5100 50  0001 C CNN
-F 3 "~" H 5400 5100 50  0001 C CNN
-F 4 "C49678" H 5400 5100 50  0001 C CNN "LCSC"
-	1    5400 5100
-	1    0    0    -1
-$EndComp
-$Comp
-L Device:C_Small C7
-U 1 1 613F7665
-P 5400 4700
-F 0 "C7" H 5492 4746 50  0000 L CNN
-F 1 "0.1uF" H 5492 4655 50  0000 L CNN
-F 2 "Capacitor_SMD:C_0805_2012Metric" H 5400 4700 50  0001 C CNN
-F 3 "~" H 5400 4700 50  0001 C CNN
-F 4 "C49678" H 5400 4700 50  0001 C CNN "LCSC"
-	1    5400 4700
-	1    0    0    -1
-$EndComp
-Connection ~ 5400 5000
-Wire Wire Line
-	5400 5000 5600 5000
-Connection ~ 5400 4800
-Wire Wire Line
-	5400 4800 5600 4800
-Wire Wire Line
-	5400 4600 5250 4600
-Wire Wire Line
-	5250 4600 5250 4900
-Connection ~ 5250 4900
-Wire Wire Line
-	5250 4900 5600 4900
-Wire Wire Line
-	5400 5200 5250 5200
-Wire Wire Line
-	5250 5200 5250 4900
-Wire Wire Line
-	5150 4800 5400 4800
-Wire Wire Line
-	5150 5000 5400 5000
-Wire Wire Line
-	5150 5200 4900 5200
-Wire Wire Line
-	5150 4600 4900 4600
-Wire Wire Line
-	4900 4600 4900 4800
-Wire Wire Line
-	5250 4900 4750 4900
-Wire Wire Line
-	4750 4800 4900 4800
-Connection ~ 4900 4800
-Wire Wire Line
-	4900 4800 4900 5200
 $EndSCHEMATC
