File: pcb/vertex.kicad_pcb (KiCad board)
At the start: 2 copper layers, 247 x 78.9 mm, 89 parts, among them U1 ATmega32U2-AU, U2 SRV05-4, X1 Crystal_GND24_Small

Commit message: finalized PCB
Parts:
- added D24: D_Small, custom_parts:D_SOT-23_ANK_norm, B.Cu at (149.7, 113.2)
- added MX46: MX-NoLED, MX_Only:MXOnly-1U-NoLED, F.Cu at (35.7, 123.0)
- added MX47: MX-NoLED, MX_Only:MXOnly-1U-NoLED, F.Cu at (54.8, 123.0)
- added MX48: MX-NoLED, MX_Only:MXOnly-1U-NoLED, F.Cu at (73.8, 123.0)
- added MX49: MX-NoLED, MX_Only:MXOnly-1U-NoLED, F.Cu at (92.9, 123.0)
- added MX50: MX-NoLED, MX_Only:MXOnly-1U-NoLED, F.Cu at (207.2, 123.0)
- added MX51: MX-NoLED, MX_Only:MXOnly-1U-NoLED, F.Cu at (226.2, 123.0)
- added MX52: MX-NoLED, MX_Only:MXOnly-1U-NoLED, F.Cu at (245.3, 123.0)
- added MX53: MX-NoLED, MX_Only:MXOnly-1U-NoLED, F.Cu at (264.3, 123.0)
- added MX54: MX-NoLED, MX_Only:MXOnly-2.75U-ReversedStabilizers-NoLED, F.Cu at (171.4, 123.0)
- added MX55: MX-NoLED, MX_Only:MXOnly-2.25U-ReversedStabilizers-NoLED, F.Cu at (123.8, 123.0)
- added MX60: MX-NoLED, MX_Only:MXOnly-2U-NoLED, F.Cu at (254.8, 65.9)
- added MX66: MX-NoLED, MX_Only:MXOnly-1.25U-NoLED, F.Cu at (242.9, 104.0)
- added MX67: MX-NoLED, MX_Only:MXOnly-1U-NoLED, F.Cu at (264.3, 104.0)
- D1, D10, D11, D12, D13, D14, D15, D16, D17, D18, D19, D2, D20, D21, D22, D23, D3, D4, D5, D6, D7, D8, D9: footprint custom_parts:D_SOT-23_ANK -> custom_parts:D_SOT-23_ANK_norm
- moved D21 25.9 mm to (82.8, 113.2), turned to 90 degrees
- moved D22 25.2 mm to (219.6, 113.2), turned to 90 degrees
- moved D23 15.6 mm to (254.8, 113.2), turned to 90 degrees
- moved D20 13.0 mm to (50.7, 113.2), turned to 90 degrees
- moved D7 3.94 mm to (254.8, 72.6)
- moved D19 2.16 mm to (252.2, 107.6)
Connections:
- MX10 pad 2: Net-(D5-Pad2) -> Net-(D5-Pad3)
- MX12 pad 2: Net-(D6-Pad2) -> Net-(D6-Pad3)
- MX13 pad 2: Net-(D7-Pad2) -> Net-(D7-Pad3)
- MX14 pad 2: Net-(D8-Pad2) -> Net-(D8-Pad3)
- MX17 pad 2: Net-(D9-Pad2) -> Net-(D9-Pad3)
- MX19 pad 2: Net-(D10-Pad2) -> Net-(D10-Pad3)
- MX2 pad 2: Net-(D1-Pad2) -> Net-(D1-Pad3)
- MX21 pad 2: Net-(D11-Pad2) -> Net-(D11-Pad3)
- MX23 pad 2: Net-(D12-Pad2) -> Net-(D12-Pad3)
- MX25 pad 2: Net-(D13-Pad2) -> Net-(D13-Pad3)
- MX27 pad 2: Net-(D14-Pad2) -> Net-(D14-Pad3)
- MX29 pad 2: Net-(D15-Pad2) -> Net-(D15-Pad3)
- MX31 pad 2: Net-(D16-Pad2) -> Net-(D16-Pad3)
- MX33 pad 2: Net-(D17-Pad2) -> Net-(D17-Pad3)
- MX35 pad 2: Net-(D18-Pad2) -> Net-(D18-Pad3)
- MX37 pad 2: Net-(D19-Pad2) -> Net-(D19-Pad3)
- MX38 pad 2: Net-(D20-Pad2) -> Net-(D20-Pad3)
- MX39 pad 1: col1 -> col2
- MX39 pad 2: Net-(D20-Pad2) -> Net-(D21-Pad3)
- MX4 pad 2: Net-(D2-Pad2) -> Net-(D2-Pad3)
- MX40 pad 1: col2 -> col3
- MX41 pad 2: Net-(D21-Pad2) -> Net-(D24-Pad3)
- MX42 pad 1: col7 -> col6
- MX42 pad 2: Net-(D22-Pad2) -> Net-(D24-Pad2)
- MX43 pad 1: col8 -> col7
- MX43 pad 2: Net-(D22-Pad2) -> Net-(D22-Pad3)
- MX44 pad 1: col9 -> col8
- MX44 pad 2: Net-(D23-Pad2) -> Net-(D22-Pad2)
- MX6 pad 2: Net-(D3-Pad2) -> Net-(D3-Pad3)
- MX8 pad 2: Net-(D4-Pad2) -> Net-(D4-Pad3)
Routing:
- net row3: track 309.2 -> 273.6 mm, vias 0 -> 2
- net Net-(D24-Pad3): track 0.00 -> 34.6 mm
- net Net-(D24-Pad2): track 0.00 -> 34.1 mm
- net Net-(D21-Pad2): track 45.9 -> 13.2 mm
- net col3: track 81.1 -> 112.0 mm
- net col6: track 138.3 -> 166.6 mm
- net col10: track 245.7 -> 272.8 mm
- net Net-(D20-Pad2): track 33.9 -> 7.05 mm
- net Net-(D6-Pad3): track 0.00 -> 25.9 mm
- net Net-(D13-Pad3): track 0.00 -> 23.9 mm
- net Net-(D13-Pad2): track 35.6 -> 11.7 mm
- net Net-(D23-Pad2): track 34.1 -> 11.3 mm
- net Net-(D20-Pad3): track 0.00 -> 22.6 mm
- net col8: track 197.0 -> 217.6 mm
- net Net-(D7-Pad3): track 0.00 -> 20.4 mm
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
Commit message: finalize repo layout
Parts:
- renumbered C6 to C4, C7 to C5, C5 to C6

Commit message: update gerbers
Routing:
- net GND: track 31.5 -> 31.4 mm, vias 1 -> 2
Changed lines of the file:
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@@
       (drillshape 0)
       (scaleselection 1)
-      (outputdirectory ""))
+      (outputdirectory "gerbers"))
   )
   (net 0 "")
@@
   (segment (start 54.032686 99.441) (end 51.181 99.441) (width 0.5) (layer B.Cu) (net 1))
   (via (at 66.802 91.313) (size 0.8) (drill 0.4) (layers F.Cu B.Cu) (net 1))
-  (segment (start 66.421 90.932) (end 66.802 91.313) (width 0.5) (layer B.Cu) (net 1))
-  (segment (start 65.3015 90.932) (end 66.421 90.932) (width 0.5) (layer B.Cu) (net 1))
+  (segment (start 65.3015 90.932) (end 66.802 91.313) (width 0.5) (layer B.Cu) (net 1))
+  (via (at 57.3405 95.5675) (size 0.8) (drill 0.4) (layers F.Cu B.Cu) (net 1))
   (segment (start 45.974 80.01) (end 47.3075 78.6765) (width 0.5) (layer B.Cu) (net 2))
   (segment (start 47.3075 78.6765) (end 48.7045 78.6765) (width 0.5) (layer B.Cu) (net 2))
